File: quad-ref-clock.sch (EAGLE design)
At the start: 31 parts, among them U1 LMK00804B, U2 ADP150, U3 ADP150, X1 SMA, X2 SMA, X3 SMA, X4 SMA

Commit message: update
Parts:
- removed R5: 49.9, rcl:R-US_R0805
- added R4: 49.9, rcl:R-US_R0603
Connections:
- net GND: now also R4.1; no longer R5.1
- net N$7: now also R4.2; no longer R5.2
Changed lines of the file:
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@@
 <setting verticaltext="up"/>
 </settings>
-<grid distance="0.1" unitdist="inch" unit="inch" style="lines" multiple="1" display="no" altdistance="0.01" altunitdist="inch" altunit="inch"/>
+<grid distance="0.05" unitdist="inch" unit="inch" style="lines" multiple="1" display="yes" altdistance="0.01" altunitdist="inch" altunit="inch"/>
 <layers>
 <layer number="1" name="Top" color="4" fill="1" visible="no" active="no"/>
@@
 <part name="P+1" library="supply1" deviceset="VCC" device=""/>
 <part name="P+2" library="supply1" deviceset="VCC" device=""/>
-<part name="R5" library="rcl" deviceset="R-US_" device="R0805" value="49.9"/>
 <part name="GND7" library="supply1" deviceset="GND" device=""/>
 <part name="C4" library="rcl" deviceset="C-EU" device="C0805" value="100n"/>
@@
 <part name="X4" library="con-coax" deviceset="SMA-" device="142-0711-881/886" value="SMA"/>
 <part name="R3" library="rcl" deviceset="R-US_" device="R0805" value="1k"/>
+<part name="R4" library="rcl" deviceset="R-US_" device="R0603" value="49.9"/>
 </parts>
 <sheets>
@@
 </instance>
 <instance part="P+2" gate="VCC" x="93.98" y="121.92"/>
-<instance part="R5" gate="G$1" x="93.98" y="88.9" rot="R90"/>
 <instance part="GND7" gate="1" x="93.98" y="81.28"/>
 <instance part="C4" gate="G$1" x="170.18" y="157.48" rot="R90"/>
@@
 <instance part="X4" gate="G1" x="208.28" y="101.6" rot="MR0"/>
 <instance part="R3" gate="G$1" x="109.22" y="101.6"/>
+<instance part="R4" gate="G$1" x="93.98" y="88.9" rot="R90"/>
 </instances>
 <busses>
@@
 <pinref part="U1" gate="G$1" pin="LVCMOS_CLK"/>
 <wire x1="114.3" y1="96.52" x2="93.98" y2="96.52" width="0.1524" layer="91"/>
-<pinref part="R5" gate="G$1" pin="2"/>
 <wire x1="93.98" y1="93.98" x2="93.98" y2="96.52" width="0.1524" layer="91"/>
 <pinref part="C3" gate="G$1" pin="2"/>
 <wire x1="85.09" y1="96.52" x2="93.98" y2="96.52" width="0.1524" layer="91"/>
 <junction x="93.98" y="96.52"/>
+<pinref part="R4" gate="G$1" pin="2"/>
 </segment>
 </net>
@@
 </segment>
 <segment>
-<pinref part="R5" gate="G$1" pin="1"/>
-<pinref part="GND7" gate="1" pin="GND"/>
-</segment>
-<segment>
 <pinref part="C4" gate="G$1" pin="1"/>
 <wire x1="167.64" y1="157.48" x2="165.1" y2="154.94" width="0.1524" layer="91"/>
@@
 <pinref part="GND20" gate="1" pin="GND"/>
 </segment>
+<segment>
+<pinref part="GND7" gate="1" pin="GND"/>
+<pinref part="R4" gate="G$1" pin="1"/>
+</segment>
 </net>

Commit message: update
Parts:
- removed R9: 43, rcl:R-US_R0805
- added R5: 43, rcl:R-US_R0603
- R6, R7, R8: device rcl:R-US_R0805 -> rcl:R-US_R0603
Connections:
- net N$1: now also R5.1; no longer R6.1
- net N$10: now also R5.2; no longer R6.2
- net N$11: now also R6.2; no longer R7.2
- net N$12: now also R7.2; no longer R8.2
- net N$13: now also R8.2; no longer R9.2
- net N$2: now also R6.1; no longer R7.1
- net N$3: now also R7.1; no longer R8.1
- net N$4: now also R8.1; no longer R9.1
Other:
- moved on the sheet: R6, R7, R8
Changed lines of the file:
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@@
 <setting verticaltext="up"/>
 </settings>
-<grid distance="0.05" unitdist="inch" unit="inch" style="lines" multiple="1" display="yes" altdistance="0.01" altunitdist="inch" altunit="inch"/>
+<grid distance="0.1" unitdist="inch" unit="inch" style="lines" multiple="1" display="no" altdistance="0.01" altunitdist="inch" altunit="inch"/>
 <layers>
 <layer number="1" name="Top" color="4" fill="1" visible="no" active="no"/>
@@
 <part name="C5" library="rcl" deviceset="C-EU" device="C0805" value="100n"/>
 <part name="GND9" library="supply1" deviceset="GND" device=""/>
-<part name="R6" library="rcl" deviceset="R-US_" device="R0805" value="43"/>
-<part name="R7" library="rcl" deviceset="R-US_" device="R0805" value="43"/>
-<part name="R8" library="rcl" deviceset="R-US_" device="R0805" value="43"/>
-<part name="R9" library="rcl" deviceset="R-US_" device="R0805" value="43"/>
 <part name="GND12" library="supply1" deviceset="GND" device=""/>
 <part name="C3" library="rcl" deviceset="C-EU" device="C0805" value="470pF"/>
@@
 <part name="R3" library="rcl" deviceset="R-US_" device="R0805" value="1k"/>
 <part name="R4" library="rcl" deviceset="R-US_" device="R0603" value="49.9"/>
+<part name="R5" library="rcl" deviceset="R-US_" device="R0603" value="43"/>
+<part name="R6" library="rcl" deviceset="R-US_" device="R0603" value="43"/>
+<part name="R7" library="rcl" deviceset="R-US_" device="R0603" value="43"/>
+<part name="R8" library="rcl" deviceset="R-US_" device="R0603" value="43"/>
 </parts>
 <sheets>
@@
 <instance part="C5" gate="G$1" x="195.58" y="157.48" rot="R90"/>
 <instance part="GND9" gate="1" x="190.5" y="152.4"/>
-<instance part="R6" gate="G$1" x="177.8" y="132.08"/>
-<instance part="R7" gate="G$1" x="177.8" y="121.92"/>
-<instance part="R8" gate="G$1" x="177.8" y="111.76"/>
-<instance part="R9" gate="G$1" x="177.8" y="101.6"/>
 <instance part="GND12" gate="1" x="43.18" y="81.28"/>
 <instance part="C3" gate="G$1" x="80.01" y="96.52" rot="R90"/>
@@
 <instance part="R3" gate="G$1" x="109.22" y="101.6"/>
 <instance part="R4" gate="G$1" x="93.98" y="88.9" rot="R90"/>
+<instance part="R5" gate="G$1" x="177.8" y="132.08"/>
+<instance part="R6" gate="G$1" x="177.8" y="121.92"/>
+<instance part="R7" gate="G$1" x="177.8" y="111.76"/>
+<instance part="R8" gate="G$1" x="177.8" y="101.6"/>
 </instances>
 <busses>
@@
 <segment>
 <pinref part="U1" gate="G$1" pin="Q0"/>
+<wire x1="154.94" y1="132.08" x2="172.72" y2="132.08" width="0.1524" layer="91"/>
+<pinref part="R5" gate="G$1" pin="1"/>
+</segment>
+</net>
+<net name="N$2" class="0">
+<segment>
+<pinref part="U1" gate="G$1" pin="Q1"/>
+<wire x1="154.94" y1="121.92" x2="172.72" y2="121.92" width="0.1524" layer="91"/>
 <pinref part="R6" gate="G$1" pin="1"/>
-<wire x1="154.94" y1="132.08" x2="172.72" y2="132.08" width="0.1524" layer="91"/>
-</segment>
-</net>
-<net name="N$2" class="0">
-<segment>
-<pinref part="U1" gate="G$1" pin="Q1"/>
+</segment>
+</net>
+<net name="N$3" class="0">
+<segment>
+<pinref part="U1" gate="G$1" pin="Q2"/>
+<wire x1="154.94" y1="111.76" x2="172.72" y2="111.76" width="0.1524" layer="91"/>
 <pinref part="R7" gate="G$1" pin="1"/>
-<wire x1="154.94" y1="121.92" x2="172.72" y2="121.92" width="0.1524" layer="91"/>
-</segment>
-</net>
-<net name="N$3" class="0">
-<segment>
-<pinref part="U1" gate="G$1" pin="Q2"/>
+</segment>
+</net>
+<net name="N$4" class="0">
+<segment>
+<pinref part="U1" gate="G$1" pin="Q3"/>
+<wire x1="154.94" y1="101.6" x2="172.72" y2="101.6" width="0.1524" layer="91"/>
 <pinref part="R8" gate="G$1" pin="1"/>
-<wire x1="154.94" y1="111.76" x2="172.72" y2="111.76" width="0.1524" layer="91"/>
-</segment>
-</net>
-<net name="N$4" class="0">
-<segment>
-<pinref part="U1" gate="G$1" pin="Q3"/>
-<pinref part="R9" gate="G$1" pin="1"/>
-<wire x1="154.94" y1="101.6" x2="172.72" y2="101.6" width="0.1524" layer="91"/>
 </segment>
 </net>
 <net name="N$10" class="0">
 <segment>
-<pinref part="R6" gate="G$1" pin="2"/>
 <wire x1="182.88" y1="132.08" x2="205.74" y2="132.08" width="0.1524" layer="91"/>
 <pinref part="X1" gate="G1" pin="1"/>
+<pinref part="R5" gate="G$1" pin="2"/>
 </segment>
 </net>
 <net name="N$11" class="0">
 <segment>
-<pinref part="R7" gate="G$1" pin="2"/>
 <wire x1="182.88" y1="121.92" x2="205.74" y2="121.92" width="0.1524" layer="91"/>
 <pinref part="X2" gate="G1" pin="1"/>
+<pinref part="R6" gate="G$1" pin="2"/>
 </segment>
 </net>
 <net name="N$12" class="0">
 <segment>
-<pinref part="R8" gate="G$1" pin="2"/>
 <wire x1="182.88" y1="111.76" x2="205.74" y2="111.76" width="0.1524" layer="91"/>
 <pinref part="X3" gate="G1" pin="1"/>
+<pinref part="R7" gate="G$1" pin="2"/>
 </segment>
 </net>
 <net name="N$13" class="0">
 <segment>
-<pinref part="R9" gate="G$1" pin="2"/>
 <wire x1="182.88" y1="101.6" x2="205.74" y2="101.6" width="0.1524" layer="91"/>
 <pinref part="X4" gate="G1" pin="1"/>
-</segment>
-</net>
+<pinref part="R8" gate="G$1" pin="2"/>
+</segment>
+</net>
