File: quad-ref-clock.brd (EAGLE design)
At the start: 48 x 48 mm, 29 parts, among them U1 LMK00804B, U2 ADP150, U3 ADP150, X1 SMA, X2 SMA, X3 SMA, X4 SMA

Commit message: update
Parts:
- moved R1 0.32 mm to (17.5, 21.9)
- turned R5 to 216 degrees
Routing:
- net VCC: track 47.2 -> 54.8 mm
- net N$15: track 13.9 -> 10.1 mm, vias 1 -> 0
- net GND: vias 55 -> 8
Changed lines of the file:
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@@
 <wire x1="47.495" y1="48" x2="-0.505" y2="48" width="0" layer="20"/>
 <wire x1="-0.505" y1="48" x2="-0.505" y2="0" width="0" layer="20"/>
-<text x="23.495" y="43.815" size="1.4224" layer="1" font="vector" ratio="9" align="center">Jerome ODIER</text>
+<text x="23.495" y="46.355" size="1.4224" layer="1" font="vector" ratio="9" align="center">Jerome ODIER</text>
 </plain>
 <attributes>
@@
 <attribute name="OC_FARNELL" value="unknown" x="34.29" y="8.89" size="1.778" layer="27" display="off"/>
 </element>
-<element name="R1" library="rcl" package="R0805" value="1k" x="17.465" y="22.225" rot="R90"/>
+<element name="R1" library="rcl" package="R0805" value="1k" x="17.465" y="21.9075" rot="R90"/>
 <element name="R2" library="rcl" package="R0805" value="1k" x="23.17" y="25.4"/>
-<element name="R5" library="rcl" package="R0805" value="49.9" x="30.1625" y="28.194" rot="R215"/>
+<element name="R5" library="rcl" package="R0805" value="49.9" x="30.1625" y="28.194" rot="R216"/>
 <element name="R6" library="rcl" package="R0805" value="43" x="7.62" y="39.37" rot="R180"/>
 <element name="R7" library="rcl" package="R0805" value="43" x="7.62" y="26.67" rot="R180"/>
@@
 <contactref element="R5" pad="2"/>
 <contactref element="C3" pad="2"/>
-<wire x1="34.34011875" y1="21.957609375" x2="29.384303125" y2="27.6491" width="0.4064" layer="1"/>
-<wire x1="29.384303125" y1="27.6491" x2="25.77" y2="30.145" width="0.4064" layer="1" curve="32.15025"/>
+<wire x1="34.34011875" y1="21.957609375" x2="29.39393125" y2="27.635603125" width="0.4064" layer="1"/>
+<wire x1="29.39393125" y1="27.635603125" x2="25.77" y2="30.145" width="0.4064" layer="1" curve="32.15025"/>
 </signal>
 <signal name="GND">
@@
 <wire x1="24.384" y1="26.67" x2="27.432" y2="26.67" width="0.3048" layer="1"/>
 <via x="1.27" y="46.355" extent="1-16" drill="0.5"/>
-<via x="3.81" y="46.355" extent="1-16" drill="0.5"/>
-<via x="6.35" y="46.355" extent="1-16" drill="0.5"/>
-<via x="8.89" y="46.355" extent="1-16" drill="0.5"/>
-<via x="11.43" y="46.355" extent="1-16" drill="0.5"/>
-<via x="13.97" y="46.355" extent="1-16" drill="0.5"/>
-<via x="16.51" y="46.355" extent="1-16" drill="0.5"/>
-<via x="19.05" y="46.355" extent="1-16" drill="0.5"/>
-<via x="21.59" y="46.355" extent="1-16" drill="0.5"/>
-<via x="24.13" y="46.355" extent="1-16" drill="0.5"/>
-<via x="26.67" y="46.355" extent="1-16" drill="0.5"/>
-<via x="29.21" y="46.355" extent="1-16" drill="0.5"/>
-<via x="31.75" y="46.355" extent="1-16" drill="0.5"/>
-<via x="34.29" y="46.355" extent="1-16" drill="0.5"/>
-<via x="36.83" y="46.355" extent="1-16" drill="0.5"/>
-<via x="39.37" y="46.355" extent="1-16" drill="0.5"/>
-<via x="41.91" y="46.355" extent="1-16" drill="0.5"/>
-<via x="44.45" y="46.355" extent="1-16" drill="0.5"/>
 <via x="45.72" y="1.905" extent="1-16" drill="0.5"/>
-<via x="45.72" y="9.525" extent="1-16" drill="0.5"/>
-<via x="45.72" y="4.445" extent="1-16" drill="0.5"/>
-<via x="45.72" y="6.985" extent="1-16" drill="0.5"/>
-<via x="45.72" y="12.065" extent="1-16" drill="0.5"/>
-<via x="45.72" y="14.605" extent="1-16" drill="0.5"/>
-<via x="45.72" y="17.145" extent="1-16" drill="0.5"/>
 <via x="45.72" y="19.685" extent="1-16" drill="0.5"/>
-<via x="41.91" y="1.905" extent="1-16" drill="0.5"/>
-<via x="39.37" y="1.905" extent="1-16" drill="0.5"/>
-<via x="36.83" y="1.905" extent="1-16" drill="0.5"/>
-<via x="34.29" y="1.905" extent="1-16" drill="0.5"/>
-<via x="31.75" y="1.905" extent="1-16" drill="0.5"/>
-<via x="29.21" y="1.905" extent="1-16" drill="0.5"/>
-<via x="26.67" y="1.905" extent="1-16" drill="0.5"/>
-<via x="24.13" y="1.905" extent="1-16" drill="0.5"/>
-<via x="21.59" y="1.905" extent="1-16" drill="0.5"/>
-<via x="19.05" y="1.905" extent="1-16" drill="0.5"/>
-<via x="16.51" y="1.905" extent="1-16" drill="0.5"/>
-<via x="13.97" y="1.905" extent="1-16" drill="0.5"/>
-<via x="11.43" y="1.905" extent="1-16" drill="0.5"/>
-<via x="8.89" y="1.905" extent="1-16" drill="0.5"/>
-<via x="6.35" y="1.905" extent="1-16" drill="0.5"/>
-<via x="3.81" y="1.905" extent="1-16" drill="0.5"/>
 <via x="1.27" y="1.905" extent="1-16" drill="0.5"/>
 <via x="45.72" y="33.02" extent="1-16" drill="0.5"/>
 <via x="1.27" y="33.02" extent="1-16" drill="0.5"/>
-<via x="1.27" y="4.445" extent="1-16" drill="0.5"/>
-<via x="1.27" y="6.985" extent="1-16" drill="0.5"/>
-<via x="1.27" y="9.525" extent="1-16" drill="0.5"/>
-<via x="1.27" y="12.065" extent="1-16" drill="0.5"/>
-<via x="1.27" y="14.605" extent="1-16" drill="0.5"/>
-<via x="1.27" y="17.145" extent="1-16" drill="0.5"/>
 <via x="1.27" y="19.685" extent="1-16" drill="0.5"/>
-<via x="44.45" y="1.905" extent="1-16" drill="0.5"/>
 <via x="45.72" y="46.355" extent="1-16" drill="0.5"/>
-<via x="38.1" y="5.08" extent="1-16" drill="0.8"/>
 </signal>
 <signal name="N$5">
@@
 <wire x1="26.67" y1="16.4998" x2="26.6802" y2="17.145" width="0.4064" layer="1"/>
 <contactref element="QG2" pad="1"/>
-<wire x1="26.67" y1="12.7" x2="26.67" y2="5.08" width="0.4064" layer="1"/>
 <wire x1="22.22" y1="27.94" x2="22.22" y2="28.824" width="0.4064" layer="1"/>
 <wire x1="22.22" y1="27.94" x2="22.22" y2="25.4" width="0.4064" layer="1"/>
@@
 <wire x1="20.005" y1="17.145" x2="20.005" y2="13.3049" width="0.4064" layer="1"/>
 <wire x1="20.005" y1="13.3049" x2="20.6099" y2="12.7" width="0.4064" layer="1"/>
-<via x="30.48" y="12.7" extent="1-16" drill="0.8"/>
-<via x="30.48" y="5.08" extent="1-16" drill="0.8"/>
-<wire x1="26.67" y1="12.7" x2="30.48" y2="12.7" width="0.4064" layer="1"/>
-<wire x1="26.67" y1="5.08" x2="30.48" y2="5.08" width="0.4064" layer="1"/>
+<via x="34.29" y="12.7" extent="1-16" drill="0.8"/>
+<via x="34.29" y="5.08" extent="1-16" drill="0.8"/>
+<wire x1="26.67" y1="12.7" x2="34.29" y2="12.7" width="0.4064" layer="1"/>
+<wire x1="34.29" y1="5.08" x2="34.29" y2="12.7" width="0.4064" layer="1"/>
+<wire x1="26.67" y1="5.08" x2="26.67" y2="12.7" width="0.4064" layer="1"/>
 <wire x1="16.64" y1="11.43" x2="19.37" y2="11.4601" width="0" layer="19" extent="1-1"/>
 </signal>
@@
 <contactref element="R1" pad="2"/>
 <wire x1="21.87" y1="30.145" x2="21.87" y2="29.49" width="0.4064" layer="1"/>
-<wire x1="17.465" y1="23.175" x2="17.465" y2="25.085" width="0.4064" layer="1"/>
+<wire x1="17.465" y1="22.8575" x2="17.465" y2="25.085" width="0.4064" layer="1"/>
 <wire x1="17.465" y1="25.085" x2="21.87" y2="29.49" width="0.4064" layer="1"/>
 </signal>
@@
 <wire x1="16.8275" y1="33.9725" x2="14.9225" y2="35.2425" width="0.4064" layer="1" curve="-67.380135"/>
 <wire x1="13.0175" y1="38.1" x2="11.1125" y2="39.37" width="0.4064" layer="1" curve="45.23973"/>
-<wire x1="21.22" y1="35.895" x2="21.22" y2="35.26" width="0.4064" layer="1"/>
+<wire x1="21.22" y1="35.895" x2="21.22" y2="35.26" width="0.35" layer="1"/>
 <wire x1="19.9325" y1="33.9725" x2="21.22" y2="35.26" width="0.4064" layer="1" curve="90"/>
 </signal>
@@
 <wire x1="16.8275" y1="32.0675" x2="14.9225" y2="30.7975" width="0.4064" layer="1" curve="67.380135"/>
 <wire x1="13.0175" y1="27.94" x2="11.1125" y2="26.67" width="0.4064" layer="1" curve="-45.23973"/>
-<wire x1="22.52" y1="35.895" x2="22.52" y2="33.315" width="0.4064" layer="1"/>
 <wire x1="21.2725" y1="32.0675" x2="22.52" y2="33.315" width="0.4064" layer="1" curve="90"/>
+<wire x1="22.52" y1="35.895" x2="22.52" y2="35.26" width="0.35" layer="1"/>
+<wire x1="22.52" y1="35.26" x2="22.52" y2="33.315" width="0.4064" layer="1"/>
 </signal>
 <signal name="N$3">
@@
 <wire x1="30.1625" y1="32.0675" x2="32.0675" y2="30.7975" width="0.4064" layer="1" curve="-67.380135"/>
 <wire x1="33.9725" y1="27.94" x2="35.8775" y2="26.67" width="0.4064" layer="1" curve="45.23973"/>
-<wire x1="23.82" y1="35.895" x2="23.82" y2="33.33" width="0.4064" layer="1"/>
 <wire x1="25.0825" y1="32.0675" x2="23.82" y2="33.33" width="0.4064" layer="1" curve="-90"/>
+<wire x1="23.82" y1="35.895" x2="23.82" y2="35.26" width="0.35" layer="1"/>
+<wire x1="23.82" y1="35.26" x2="23.82" y2="33.33" width="0.4064" layer="1"/>
 </signal>
 <signal name="N$4">
@@
 <wire x1="30.1625" y1="33.9725" x2="32.0675" y2="35.2425" width="0.4064" layer="1" curve="67.380135"/>
 <wire x1="33.9725" y1="38.1" x2="35.8775" y2="39.37" width="0.4064" layer="1" curve="-45.23973"/>
-<wire x1="25.12" y1="35.895" x2="25.12" y2="35.205" width="0.4064" layer="1"/>
+<wire x1="25.12" y1="35.895" x2="25.12" y2="35.205" width="0.35" layer="1"/>
 <wire x1="26.3525" y1="33.9725" x2="25.12" y2="35.205" width="0.4064" layer="1" curve="-90"/>
 </signal>
@@
 <contactref element="QG2" pad="8"/>
 <wire x1="41.91" y1="12.7" x2="35.509878125" y2="20.4603875" width="0.4064" layer="1"/>
-<via x="38.1" y="12.7" extent="1-16" drill="0.8"/>
-<wire x1="38.1" y1="12.7" x2="41.91" y2="12.7" width="0.4064" layer="1"/>
 </signal>
 <signal name="N$16">
 <contactref element="R1" pad="1"/>
 <contactref element="JP2" pad="2"/>
-<wire x1="17.465" y1="17.145" x2="17.465" y2="21.275" width="0.4064" layer="1"/>
+<wire x1="17.465" y1="17.145" x2="17.465" y2="20.9575" width="0.4064" layer="1"/>
 </signal>
 <signal name="C2">

Commit message: update
Parts:
- removed R5: 49.9, rcl:R0805
- added R4: 49.9, rcl:R0603
- moved C3 3.28 mm to (36.8, 18.5), turned to 129 degrees
- moved C4 0.25 mm to (22.2, 39.1)
- moved C5 0.25 mm to (24.8, 39.1)
- moved R3 0.25 mm to (26.2, 26.7)
Connections:
- net GND: now also R4.1; no longer R5.1
- net N$7: now also R4.2; no longer R5.2
Routing:
- net GND: track 3.05 -> 10.9 mm, vias 8 -> 22
- net N$7: track 11.9 -> 16.9 mm
- net N$15: track 10.1 -> 6.79 mm
- net VCC: track 54.8 -> 57.5 mm
- net VDDO: track 45.8 -> 43.2 mm

Commit message: update
Parts:
- removed R9: 43, rcl:R0805
- added R5: 43, rcl:R0603
- R6, R7, R8: device rcl:R0805 -> rcl:R0603
- moved R7 21.6 mm to (28.6, 32.1), turned to 0 degrees
- moved R6 13.0 mm to (18.4, 32.1)
- moved R8 13.0 mm to (28.6, 34.0)
- moved C2 1.91 mm to (27.6, 17.1), turned to 180 degrees
Connections:
- net N$1: now also R5.1; no longer R6.1
- net N$10: now also R5.2; no longer R6.2
- net N$11: now also R6.2; no longer R7.2
- net N$12: now also R7.2; no longer R8.2
- net N$13: now also R8.2; no longer R9.2
- net N$2: now also R6.1; no longer R7.1
- net N$3: now also R7.1; no longer R8.1
- net N$4: now also R8.1; no longer R9.1
Routing:
- net N$3: track 20.0 -> 7.29 mm
- net N$4: track 16.8 -> 4.18 mm
- net N$2: track 19.3 -> 6.72 mm
- net N$11: track 4.10 -> 16.6 mm
- net N$12: track 4.10 -> 16.6 mm
- net N$10: track 4.10 -> 16.6 mm
- net N$13: track 4.10 -> 16.6 mm
- net N$1: track 16.1 -> 3.61 mm
- net VCC: track 57.5 -> 65.2 mm
- net GND: track 10.9 -> 8.81 mm, vias 22 -> 23

Commit message: update
Parts:
- moved X3 1.27 mm to (45.7, 26.7)
- moved X4 1.27 mm to (45.7, 39.4)
- moved C1 0.64 mm to (22.5, 27.9)
- moved C2 0.64 mm to (27.0, 17.1)
- moved C4 0.64 mm to (21.6, 39.1)
- moved C5 0.64 mm to (24.1, 39.1)
- moved R2 0.64 mm to (22.5, 25.4)
- moved R4 0.64 mm to (27.3, 30.1)
- moved U1 0.64 mm to (22.9, 33.0)
- moved QG2 0.63 mm to (33.7, 8.89)
- moved R3 0.63 mm to (25.5, 26.7)
- moved R5 0.63 mm to (17.8, 34.0)
- moved R6 0.63 mm to (17.8, 32.1)
- moved R7 0.63 mm to (27.9, 32.1)
- moved R8 0.63 mm to (27.9, 34.0)
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Routing:
- net GND: track 8.81 -> 9.85 mm, vias 23 -> 57
- net N$2: track 6.72 -> 5.94 mm
- net N$3: track 7.29 -> 6.56 mm
- net N$11: track 16.6 -> 16.0 mm
- net N$10: track 16.6 -> 16.0 mm
- net N$12: track 16.6 -> 16.0 mm
Other:
- board size 48 x 48 mm -> 46 x 48.5 mm

Commit message: update
Parts:
- moved JP2 1.90 mm to (17.1, 15.2)
- moved C3 1.50 mm to (35.6, 19.6)
- moved R4 0.64 mm to (27.9, 30.1)
- moved U1 0.32 mm to (23.2, 33.0)
- moved C5 0.32 mm to (24.4, 39.1)
- moved C4 0.32 mm to (21.9, 39.1)
- moved C1 0.32 mm to (22.9, 27.9)
- moved R2 0.32 mm to (22.9, 25.4)
- moved R3 0.32 mm to (25.8, 26.7)
- moved R1 0.14 mm to (17.1, 21.8)
Routing:
- net VCC: track 64.8 -> 62.8 mm
- net N$16: track 3.81 -> 5.57 mm
- net N$15: track 6.50 -> 8.00 mm
- net N$7: track 16.8 -> 15.4 mm
- net GND: track 9.85 -> 9.09 mm
- net N$2: track 5.94 -> 6.48 mm

Commit message: update
Parts:
- moved JP1 0.32 mm to (5.08, 4.76)
- moved C3 0.09 mm to (35.6, 19.6)
Changed lines of the file:
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@@
 <setting verticaltext="up"/>
 </settings>
-<grid distance="0.0125" unitdist="inch" unit="inch" style="lines" multiple="1" display="yes" altdistance="0.025" altunitdist="inch" altunit="inch"/>
+<grid distance="0.025" unitdist="inch" unit="inch" style="lines" multiple="1" display="yes" altdistance="0.025" altunitdist="inch" altunit="inch"/>
 <layers>
 <layer number="1" name="Top" color="4" fill="1" visible="yes" active="yes"/>
@@
 <element name="C11" library="radiotelescope" package="CAPACITOR_POL_1210" value="1u" x="5.08" y="11.43" rot="R180"/>
 <element name="C2" library="rcl" package="C0805" value="100n" x="27.0002" y="17.145" rot="R180"/>
-<element name="C3" library="rcl" package="C0805" value="470pF" x="35.6108" y="19.6342" rot="R130"/>
+<element name="C3" library="rcl" package="C0805" value="470pF" x="35.56" y="19.558" rot="R130"/>
 <element name="C4" library="rcl" package="C0805" value="100n" x="21.9075" y="39.0525" rot="R270"/>
 <element name="C5" library="rcl" package="C0805" value="100n" x="24.4475" y="39.0525" rot="R270"/>
 <element name="C8" library="radiotelescope" package="CAPACITOR_POL_1210" value="1u" x="15.24" y="8.255" rot="R180"/>
 <element name="C9" library="radiotelescope" package="CAPACITOR_POL_1210" value="1u" x="15.24" y="11.43" rot="R180"/>
-<element name="JP1" library="pinhead" package="1X02" value="" x="5.08" y="4.445" rot="R180"/>
+<element name="JP1" library="pinhead" package="1X02" value="" x="5.08" y="4.7625" rot="R180"/>
 <element name="JP2" library="jumper" package="JP2" value="" x="17.145" y="15.24" rot="R180"/>
 <element name="L1" library="rcl" package="L3216C" value="MI1206K601R−10" x="20.32" y="5.08" rot="R270"/>
@@
 <wire x1="9.1799" y1="11.43" x2="9.21" y2="11.4601" width="0.4064" layer="1"/>
 <wire x1="9.21" y1="11.4601" x2="9.2075" y2="11.4601" width="0.4064" layer="1"/>
-<wire x1="9.2075" y1="11.4601" x2="9.2075" y2="12.4714" width="0.4064" layer="1"/>
-<via x="9.2075" y="12.4714" extent="1-16" drill="0.3048"/>
+<via x="9.525" y="12.7" extent="1-16" drill="0.3048"/>
 <contactref element="C4" pad="2"/>
 <contactref element="C5" pad="2"/>
@@
 <wire x1="17.78" y1="35.56" x2="20.32" y2="38.1" width="0.4064" layer="16"/>
 <wire x1="20.32" y1="38.1" x2="20.2438" y2="38.1" width="0.4064" layer="16"/>
-<wire x1="9.2075" y1="12.4714" x2="9.2075" y2="21.9075" width="0.4064" layer="16"/>
-<wire x1="9.2075" y1="21.9075" x2="17.78" y2="30.48" width="0.4064" layer="16"/>
+<wire x1="9.525" y1="22.225" x2="17.78" y2="30.48" width="0.4064" layer="16"/>
+<wire x1="9.2075" y1="11.4601" x2="9.2075" y2="12.3825" width="0.4064" layer="1"/>
+<wire x1="9.2075" y1="12.3825" x2="9.525" y2="12.7" width="0.4064" layer="1"/>
+<wire x1="9.525" y1="12.7" x2="9.525" y2="22.225" width="0.4064" layer="16"/>
 </signal>
 <signal name="N$7">
 <contactref element="U1" pad="8"/>
 <contactref element="C3" pad="2"/>
-<wire x1="35.00015" y1="20.361940625" x2="28.4734" y2="28.1178" width="0.4826" layer="1"/>
+<wire x1="34.94935" y1="20.285740625" x2="28.4734" y2="28.1178" width="0.4826" layer="1"/>
 <contactref element="R4" pad="2"/>
 <wire x1="28.4734" y1="28.1178" x2="25.46" y2="30.145" width="0.4826" layer="1" curve="32.978915" cap="flat"/>
@@
 <contactref element="C3" pad="1"/>
 <contactref element="QG2" pad="8"/>
-<wire x1="41.275" y1="12.7" x2="36.221446875" y2="18.90645625" width="0.4826" layer="1"/>
+<wire x1="41.275" y1="12.7" x2="36.170646875" y2="18.83025625" width="0.4826" layer="1"/>
 </signal>
 <signal name="N$16">
@@
 <contactref element="JP1" pad="1"/>
 <wire x1="10.16" y1="3.58" x2="20.32" y2="3.58" width="0.6096" layer="1"/>
-<wire x1="10.16" y1="3.58" x2="7.215" y2="3.58" width="0.6096" layer="1"/>
-<wire x1="7.215" y1="3.58" x2="6.35" y2="4.445" width="0.6096" layer="1"/>
+<wire x1="10.16" y1="3.58" x2="7.5325" y2="3.58" width="0.6096" layer="1"/>
+<wire x1="7.5325" y1="3.58" x2="6.35" y2="4.7625" width="0.6096" layer="1"/>
 </signal>
 <signal name="N$14">
